Commit message: feat: add Elsipder Mini Interface

File: model/ElSpider_Mini/urdf/el_mini.urdf (robot description, URDF)
Before this commit: robot el_mini, 25 links, 24 joints
Links:
- link BASE: geometry collision mesh filename=package://fast_legged_planner/model/ElSpider_Mini/meshes/BA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; visual mesh filename=package://fast_legged_planner/model/ElSpider_Mini/meshes/BA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
- link LB_FOOT: geometry collision mesh filename=package://fast_legged_planner/model/ElSpider_Mini/meshes/LB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; visual mesh filename=package://fast_legged_planner/model/ElSpider_Mini/meshes/LB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
- link LB_HIP: geometry collision mesh filename=package://fast_legged_planner/model/ElSpider_Mini/meshes/LB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; visual mesh filename=package://fast_legged_planner/model/ElSpider_Mini/meshes/LB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
- link LB_SHANK: geometry collision mesh filename=package://fast_legged_planner/model/ElSpider_Mini/meshes/LB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; visual mesh filename=package://fast_legged_planner/model/ElSpider_Mini/meshes/LB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
- link LB_THIGH: geometry collision mesh filename=package://fast_legged_planner/model/ElSpider_Mini/meshes/LB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; visual mesh filename=package://fast_legged_planner/model/ElSpider_Mini/meshes/LB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
- link LF_FOOT: geometry collision mesh filename=package://fast_legged_planner/model/ElSpider_Mini/meshes/LF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; visual mesh filename=package://fast_legged_planner/model/ElSpider_Mini/meshes/LF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
- link LF_HIP: geometry collision mesh filename=package://fast_legged_planner/model/ElSpider_Mini/meshes/LF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; visual mesh filename=package://fast_legged_planner/model/ElSpider_Mini/meshes/LF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
- link LF_SHANK: geometry collision mesh filename=package://fast_legged_planner/model/ElSpider_Mini/meshes/LF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; visual mesh filename=package://fast_legged_planner/model/ElSpider_Mini/meshes/LF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
- link LF_THIGH: geometry collision mesh filename=package://fast_legged_planner/model/ElSpider_Mini/meshes/LF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; visual mesh filename=package://fast_legged_planner/model/ElSpider_Mini/meshes/LF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
- link LM_FOOT: geometry collision mesh filename=package://fast_legged_planner/model/ElSpider_Mini/meshes/LM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; visual mesh filename=package://fast_legged_planner/model/ElSpider_Mini/meshes/LM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
- link LM_HIP: geometry collision mesh filename=package://fast_legged_planner/model/ElSpider_Mini/meshes/LM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; visual mesh filename=package://fast_legged_planner/model/ElSpider_Mini/meshes/LM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
- link LM_SHANK: geometry collision mesh filename=package://fast_legged_planner/model/ElSpider_Mini/meshes/LM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; visual mesh filename=package://fast_legged_planner/model/ElSpider_Mini/meshes/LM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
- link LM_THIGH: geometry collision mesh filename=package://fast_legged_planner/model/ElSpider_Mini/meshes/LM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; visual mesh filename=package://fast_legged_planner/model/ElSpider_Mini/meshes/LM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
- link RB_FOOT: geometry collision mesh filename=package://fast_legged_planner/model/ElSpider_Mini/meshes/RB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; visual mesh filename=package://fast_legged_planner/model/ElSpider_Mini/meshes/RB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
- link RB_HIP: geometry collision mesh filename=package://fast_legged_planner/model/ElSpider_Mini/meshes/RB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; visual mesh filename=package://fast_legged_planner/model/ElSpider_Mini/meshes/RB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
- link RB_SHANK: geometry collision mesh filename=package://fast_legged_planner/model/ElSpider_Mini/meshes/RB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; visual mesh filename=package://fast_legged_planner/model/ElSpider_Mini/meshes/RB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
- link RB_THIGH: geometry collision mesh filename=package://fast_legged_planner/model/ElSpider_Mini/meshes/RB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; visual mesh filename=package://fast_legged_planner/model/ElSpider_Mini/meshes/RB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
- link RF_FOOT: geometry collision mesh filename=package://fast_legged_planner/model/ElSpider_Mini/meshes/RF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; visual mesh filename=package://fast_legged_planner/model/ElSpider_Mini/meshes/RF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
- link RF_HIP: geometry collision mesh filename=package://fast_legged_planner/model/ElSpider_Mini/meshes/RF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; visual mesh filename=package://fast_legged_planner/model/ElSpider_Mini/meshes/RF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
- link RF_SHANK: geometry collision mesh filename=package://fast_legged_planner/model/ElSpider_Mini/meshes/RF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; visual mesh filename=package://fast_legged_planner/model/ElSpider_Mini/meshes/RF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
- link RF_THIGH: geometry collision mesh filename=package://fast_legged_planner/model/ElSpider_Mini/meshes/RF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; visual mesh filename=package://fast_legged_planner/model/ElSpider_Mini/meshes/RF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
- link RM_FOOT: geometry collision mesh filename=package://fast_legged_planner/model/ElSpider_Mini/meshes/RM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; visual mesh filename=package://fast_legged_planner/model/ElSpider_Mini/meshes/RM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
- link RM_HIP: geometry collision mesh filename=package://fast_legged_planner/model/ElSpider_Mini/meshes/RM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; visual mesh filename=package://fast_legged_planner/model/ElSpider_Mini/meshes/RM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
- link RM_SHANK: geometry collision mesh filename=package://fast_legged_planner/model/ElSpider_Mini/meshes/RM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; visual mesh filename=package://fast_legged_planner/model/ElSpider_Mini/meshes/RM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
- link RM_THIGH: geometry collision mesh filename=package://fast_legged_planner/model/ElSpider_Mini/meshes/RM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; visual mesh filename=package://fast_legged_planner/model/ElSpider_Mini/meshes/RM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
