Commit message: refactor: rename hexapod_robot_assets to robot_assets

File: dependency/robot_assets/model/elspider_air/xacro/const.xacro (robot description, xacro)
@@ -57,4 +57,4 @@
     <xacro:arg name="organize_cloud" default="false"/>
     <xacro:property name="organize_cloud" value="$(arg organize_cloud)" />
-    <xacro:property name="mesh_path" value="file://$(find hexapod_robot_assets)/model/elspider_air/meshes"/>
+    <xacro:property name="mesh_path" value="file://$(find robot_assets)/model/elspider_air/meshes"/>
 </robot>

File: dependency/robot_assets/model/elspider_air/xacro/leg.xacro (robot description, xacro)
@@ -1,5 +1,5 @@
 <?xml version="1.0"?>
 <robot xmlns:xacro="http://www.ros.org/wiki/xacro">
-    <xacro:include filename="$(find hexapod_robot_assets)/model/elspider_air/xacro/transmission.xacro"/>
+    <xacro:include filename="$(find robot_assets)/model/elspider_air/xacro/transmission.xacro"/>
     <xacro:macro name="leg" params="name mirror back special special2 *origin">
         <!-- right mirror == 1, left mirror == -1 -->

File: dependency/robot_assets/model/elspider_air/xacro/robot.xacro (robot description, xacro)
@@ -8,8 +8,8 @@
     <xacro:arg name="sensor_module_name" default="None"/>
     <xacro:property name="sensor_module_name" value="$(arg sensor_module_name)"/>
-    <xacro:include filename="$(find hexapod_robot_assets)/model/elspider_air/xacro/const.xacro"/>
-    <xacro:include filename="$(find hexapod_robot_assets)/model/elspider_air/xacro/trunk.xacro"/>
-    <xacro:include filename="$(find hexapod_robot_assets)/model/elspider_air/xacro/leg.xacro"/>
-    <xacro:include filename="$(find hexapod_robot_assets)/model/elspider_air/xacro/gazebo.xacro"/>
+    <xacro:include filename="$(find robot_assets)/model/elspider_air/xacro/const.xacro"/>
+    <xacro:include filename="$(find robot_assets)/model/elspider_air/xacro/trunk.xacro"/>
+    <xacro:include filename="$(find robot_assets)/model/elspider_air/xacro/leg.xacro"/>
+    <xacro:include filename="$(find robot_assets)/model/elspider_air/xacro/gazebo.xacro"/>
     <xacro:if value="${sensor_module_name == 'HexPercept1'}">
         <xacro:include filename="$(find hexapod_elevation_mapping)/model/modules/HexPercept1/HexPercept1.xacro"/>

File: dependency/robot_assets/model/elspider_air/xacro/robot_index_corrected.xacro (robot description, xacro)
@@ -9,8 +9,8 @@
     <xacro:arg name="sensor_module_name" default="None"/>
     <xacro:property name="sensor_module_name" value="$(arg sensor_module_name)"/>
-    <xacro:include filename="$(find hexapod_robot_assets)/model/elspider_air/xacro/const.xacro"/>
-    <xacro:include filename="$(find hexapod_robot_assets)/model/elspider_air/xacro/trunk.xacro"/>
-    <xacro:include filename="$(find hexapod_robot_assets)/model/elspider_air/xacro/leg.xacro"/>
-    <xacro:include filename="$(find hexapod_robot_assets)/model/elspider_air/xacro/gazebo.xacro"/>
+    <xacro:include filename="$(find robot_assets)/model/elspider_air/xacro/const.xacro"/>
+    <xacro:include filename="$(find robot_assets)/model/elspider_air/xacro/trunk.xacro"/>
+    <xacro:include filename="$(find robot_assets)/model/elspider_air/xacro/leg.xacro"/>
+    <xacro:include filename="$(find robot_assets)/model/elspider_air/xacro/gazebo.xacro"/>
     <xacro:if value="${sensor_module_name == 'HexPercept1'}">
         <xacro:include filename="$(find hexapod_elevation_mapping)/model/modules/HexPercept1/HexPercept1.xacro"/>
